File: pcb-tutorial.kicad_pcb (KiCad board)
At the start: 2 copper layers, 77.8 x 38.1 mm, 24 parts, among them SW1 SW_Push, U1 ATmega32U4-AU, Y1 Crystal_GND24_Small

Commit message: Completed Tutorial
Routing:
- net COL1: track 51.1 -> 32.1 mm
- net COL0: track 31.8 -> 12.7 mm
- added copper zone on B.Cu, net GND
Other:
- board text added: "PCB Tutorial"
Changed lines of the file:
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@@
   (general
     (thickness 1.6)
-    (drawings 8)
-    (tracks 193)
+    (drawings 9)
+    (tracks 190)
     (zones 0)
     (modules 24)
@@
     (add_net VCC)
   )
-  (module Crystal:Crystal_SMD_3225-4Pin_3.2x2.5mm (layer B.Cu)
-    (at 203.2 28.575 180)
-    (descr "SMD Crystal SERIES SMD3225/4 http://www.txccrystal.com/images/pdf/7m-accuracy.pdf, 3.2x2.5mm^2 package")
-    (tags "SMD SMT crystal")
-    (attr smd)
-    (fp_text reference Y1 (at 0 2.45) (layer B.SilkS)
-      (effects (font (size 1 1) (thickness 0.15)) (justify mirror))
-    )
-    (fp_text value Crystal_GND24_Small (at 0 -2.45) (layer B.Fab)
-      (effects (font (size 1 1) (thickness 0.15)) (justify mirror))
-    )
-    (fp_text user %R (at 0 0) (layer B.Fab)
-      (effects (font (size 0.7 0.7) (thickness 0.105)) (justify mirror))
-    )
-    (fp_line (start -1.6 1.25) (end -1.6 -1.25) (layer B.Fab) (width 0.1))
-    (fp_line (start -1.6 -1.25) (end 1.6 -1.25) (layer B.Fab) (width 0.1))
-    (fp_line (start 1.6 -1.25) (end 1.6 1.25) (layer B.Fab) (width 0.1))
-    (fp_line (start 1.6 1.25) (end -1.6 1.25) (layer B.Fab) (width 0.1))
-    (fp_line (start -1.6 -0.25) (end -0.6 -1.25) (layer B.Fab) (width 0.1))
-    (fp_line (start -2 1.65) (end -2 -1.65) (layer B.SilkS) (width 0.12))
-    (fp_line (start -2 -1.65) (end 2 -1.65) (layer B.SilkS) (width 0.12))
-    (fp_line (start -2.1 1.7) (end -2.1 -1.7) (layer B.CrtYd) (width 0.05))
-    (fp_line (start -2.1 -1.7) (end 2.1 -1.7) (layer B.CrtYd) (width 0.05))
-    (fp_line (start 2.1 -1.7) (end 2.1 1.7) (layer B.CrtYd) (width 0.05))
-    (fp_line (start 2.1 1.7) (end -2.1 1.7) (layer B.CrtYd) (width 0.05))
-    (pad 4 smd rect (at -1.1 0.85 180) (size 1.4 1.2) (layers B.Cu B.Paste B.Mask)
-      (net 1 GND))
-    (pad 3 smd rect (at 1.1 0.85 180) (size 1.4 1.2) (layers B.Cu B.Paste B.Mask)
-      (net 3 "Net-(C2-Pad1)"))
-    (pad 2 smd rect (at 1.1 -0.85 180) (size 1.4 1.2) (layers B.Cu B.Paste B.Mask)
-      (net 1 GND))
-    (pad 1 smd rect (at -1.1 -0.85 180) (size 1.4 1.2) (layers B.Cu B.Paste B.Mask)
-      (net 2 "Net-(C1-Pad1)"))
-    (model ${KISYS3DMOD}/Crystal.3dshapes/Crystal_SMD_3225-4Pin_3.2x2.5mm.wrl
-      (at (xyz 0 0 0))
-      (scale (xyz 1 1 1))
-      (rotate (xyz 0 0 0))
-    )
-  )
   (module random-keyboard-parts:Molex-0548190589 (layer B.Cu)
     (at 184.15 23.01875 270)
@@
       (net 1 GND))
   )
+  (module Crystal:Crystal_SMD_3225-4Pin_3.2x2.5mm (layer B.Cu)
+    (at 203.2 28.575 180)
+    (descr "SMD Crystal SERIES SMD3225/4 http://www.txccrystal.com/images/pdf/7m-accuracy.pdf, 3.2x2.5mm^2 package")
+    (tags "SMD SMT crystal")
+    (attr smd)
+    (fp_text reference Y1 (at 0 2.45) (layer B.SilkS)
+      (effects (font (size 1 1) (thickness 0.15)) (justify mirror))
+    )
+    (fp_text value Crystal_GND24_Small (at 0 -2.45) (layer B.Fab)
+      (effects (font (size 1 1) (thickness 0.15)) (justify mirror))
+    )
+    (fp_text user %R (at 0 0) (layer B.Fab)
+      (effects (font (size 0.7 0.7) (thickness 0.105)) (justify mirror))
+    )
+    (fp_line (start -1.6 1.25) (end -1.6 -1.25) (layer B.Fab) (width 0.1))
+    (fp_line (start -1.6 -1.25) (end 1.6 -1.25) (layer B.Fab) (width 0.1))
+    (fp_line (start 1.6 -1.25) (end 1.6 1.25) (layer B.Fab) (width 0.1))
+    (fp_line (start 1.6 1.25) (end -1.6 1.25) (layer B.Fab) (width 0.1))
+    (fp_line (start -1.6 -0.25) (end -0.6 -1.25) (layer B.Fab) (width 0.1))
+    (fp_line (start -2 1.65) (end -2 -1.65) (layer B.SilkS) (width 0.12))
+    (fp_line (start -2 -1.65) (end 2 -1.65) (layer B.SilkS) (width 0.12))
+    (fp_line (start -2.1 1.7) (end -2.1 -1.7) (layer B.CrtYd) (width 0.05))
+    (fp_line (start -2.1 -1.7) (end 2.1 -1.7) (layer B.CrtYd) (width 0.05))
+    (fp_line (start 2.1 -1.7) (end 2.1 1.7) (layer B.CrtYd) (width 0.05))
+    (fp_line (start 2.1 1.7) (end -2.1 1.7) (layer B.CrtYd) (width 0.05))
+    (pad 4 smd rect (at -1.1 0.85 180) (size 1.4 1.2) (layers B.Cu B.Paste B.Mask)
+      (net 1 GND))
+    (pad 3 smd rect (at 1.1 0.85 180) (size 1.4 1.2) (layers B.Cu B.Paste B.Mask)
+      (net 3 "Net-(C2-Pad1)"))
+    (pad 2 smd rect (at 1.1 -0.85 180) (size 1.4 1.2) (layers B.Cu B.Paste B.Mask)
+      (net 1 GND))
+    (pad 1 smd rect (at -1.1 -0.85 180) (size 1.4 1.2) (layers B.Cu B.Paste B.Mask)
+      (net 2 "Net-(C1-Pad1)"))
+    (model ${KISYS3DMOD}/Crystal.3dshapes/Crystal_SMD_3225-4Pin_3.2x2.5mm.wrl
+      (at (xyz 0 0 0))
+      (scale (xyz 1 1 1))
+      (rotate (xyz 0 0 0))
+    )
+  )
   (module Package_QFP:TQFP-44_10x10mm_P0.8mm (layer B.Cu)
     (at 203.99375 42.8625)
@@
       (rotate (xyz 0 0 0))
     )
+  )
+  (gr_text "PCB Tutorial" (at 204.7875 57.15) (layer F.SilkS)
+    (effects (font (size 1 1) (thickness 0.15)))
   )
   (gr_line (start 177.8 59.53125) (end 250.825 59.53125) (layer Edge.Cuts) (width 0.05))
@@
   (segment (start 217.0175 43.6625) (end 220.82125 47.46625) (width 0.254) (layer B.Cu) (net 13))
   (segment (start 209.69375 43.6625) (end 217.0175 43.6625) (width 0.254) (layer B.Cu) (net 13))
-  (segment (start 220.82125 30.7975) (end 220.82125 47.46625) (width 0.254) (layer F.Cu) (net 13))
-  (segment (start 220.82125 28.41625) (end 220.82125 30.7975) (width 0.254) (layer F.Cu) (net 13))
   (segment (start 235.2675 42.8625) (end 239.87125 47.46625) (width 0.254) (layer B.Cu) (net 14))
   (segment (start 209.69375 42.8625) (end 235.2675 42.8625) (width 0.254) (layer B.Cu) (net 14))
-  (segment (start 239.87125 28.41625) (end 239.87125 47.46625) (width 0.254) (layer F.Cu) (net 14))
   (segment (start 200.79375 36.348898) (end 200.79375 37.1625) (width 0.254) (layer B.Cu) (net 15))
   (segment (start 200.530351 36.085499) (end 200.79375 36.348898) (width 0.254) (layer B.Cu) (net 15))
@@
   (segment (start 209.84375 46.7125) (end 209.69375 46.8625) (width 0.254) (layer B.Cu) (net 20))
   (segment (start 212.725 46.7125) (end 209.84375 46.7125) (width 0.254) (layer B.Cu) (net 20))
+  (zone (net 1) (net_name GND) (layer B.Cu) (hatch edge 0.508)
+    (connect_pads (clearance 0.508))
+    (min_thickness 0.254)
+    (fill yes (arc_segments 32) (thermal_gap 0.508) (thermal_bridge_width 0.508))
+    (polygon
+      (pts
+        (xy 215.10625 59.53125) (xy 177.00625 59.53125) (xy 177.00625 21.43125) (xy 215.10625 21.43125)
+      )
+    )
+  )
 )
